Commit message: 22

File: vicpinky-project-tuning/vicpinky_description/urdf/camera.xacro (robot description, xacro)
@@ -7,5 +7,5 @@
             <update_rate>30</update_rate>
             <topic>camera/image_raw</topic>
-            <gz_frame_id>camera_rgb_frame</gz_frame_id>
+            <frame>camera_rgb_frame</frame>
             <camera name="intel_realsense_r200">
                 <camera_info_topic>camera/camera_info</camera_info_topic>

File: vicpinky-project-tuning/vicpinky_description/urdf/lidar.xacro (robot description, xacro)
@@ -10,5 +10,5 @@
             <update_rate>5</update_rate>
             <topic>${prefix}scan</topic>
-            <gz_frame_id>${prefix}laser_link</gz_frame_id>
+            <frame>${prefix}laser_link</frame>
             <lidar>
                 <scan>

File: vicpinky-project-tuning/vicpinky_description/urdf/robot_core.xacro (robot description, xacro)
@@ -88,5 +88,11 @@
         </xacro:inertial_box>
     </link>
-    <link name="${prefix}base_footprint"/>
+    <link name="${prefix}base_footprint">
+        <inertial>
+            <mass value="0.001"/>
+            <origin xyz="0 0 0"/>
+            <inertia ixx="0.0001" ixy="0.0" ixz="0.0" iyy="0.0001" iyz="0.0" izz="0.0001"/>
+        </inertial>
+    </link>
     <joint name="${prefix}base_link_fixed_joint" type="fixed">
         <parent link="${prefix}base_footprint"/>
@@ -229,5 +235,11 @@
         <origin xyz="0 0 0.18" rpy="0 0 0"/>
     </joint>
-    <link name="${prefix}laser_link"/>
+    <link name="${prefix}laser_link">
+        <inertial>
+            <mass value="0.001"/>
+            <origin xyz="0 0 0"/>
+            <inertia ixx="0.0001" ixy="0.0" ixz="0.0" iyy="0.0001" iyz="0.0" izz="0.0001"/>
+        </inertial>
+    </link>
     <joint name="${prefix}laser_link_fixed_joint" type="fixed">
         <parent link="${prefix}lidar_mount"/>

Commit message: 20251106

File: vicpinky-project-tuning/vicpinky_description/urdf/camera.xacro (robot description, xacro)
@@ -7,5 +7,5 @@
             <update_rate>30</update_rate>
             <topic>camera/image_raw</topic>
-            <frame>camera_rgb_frame</frame>
+            <gz_frame_id>camera_rgb_frame</gz_frame_id>
             <camera name="intel_realsense_r200">
                 <camera_info_topic>camera/camera_info</camera_info_topic>

File: vicpinky-project-tuning/vicpinky_description/urdf/gazebo_control.xacro (robot description, xacro)
@@ -21,5 +21,5 @@
         </plugin>
         <plugin filename="gz-sim-joint-state-publisher-system" name="gz::sim::systems::JointStatePublisher">
-            <topic>${prefix}joint_states</topic>
+            <topic>joint_states</topic>
             <joint_name>${prefix}left_wheel_joint</joint_name>
             <joint_name>${prefix}right_wheel_joint</joint_name>

File: vicpinky-project-tuning/vicpinky_description/urdf/lidar.xacro (robot description, xacro)
@@ -10,5 +10,5 @@
             <update_rate>5</update_rate>
             <topic>${prefix}scan</topic>
-            <frame>${prefix}laser_link</frame>
+            <gz_frame_id>${prefix}laser_link</gz_frame_id>
             <lidar>
                 <scan>

File: vicpinky-project-tuning/vicpinky_description/urdf/robot_core.xacro (robot description, xacro)
@@ -88,11 +88,5 @@
         </xacro:inertial_box>
     </link>
-    <link name="${prefix}base_footprint">
-        <inertial>
-            <mass value="0.001"/>
-            <origin xyz="0 0 0"/>
-            <inertia ixx="0.0001" ixy="0.0" ixz="0.0" iyy="0.0001" iyz="0.0" izz="0.0001"/>
-        </inertial>
-    </link>
+    <link name="${prefix}base_footprint"/>
     <joint name="${prefix}base_link_fixed_joint" type="fixed">
         <parent link="${prefix}base_footprint"/>
@@ -235,11 +229,5 @@
         <origin xyz="0 0 0.18" rpy="0 0 0"/>
     </joint>
-    <link name="${prefix}laser_link">
-        <inertial>
-            <mass value="0.001"/>
-            <origin xyz="0 0 0"/>
-            <inertia ixx="0.0001" ixy="0.0" ixz="0.0" iyy="0.0001" iyz="0.0" izz="0.0001"/>
-        </inertial>
-    </link>
+    <link name="${prefix}laser_link"/>
     <joint name="${prefix}laser_link_fixed_joint" type="fixed">
         <parent link="${prefix}lidar_mount"/>
